File: hardware/Pajoniiir-M1/06_USB_POWER.kicad_sch (KiCad schematic)
At the start: 0 parts

Commit message: hardware: capture independent dual USB VBUS power
Parts:
- added C_USB0_IN, C_USB0_OUT_HF, C_USB1_IN, C_USB1_OUT_HF: 100nF, Capacitor_SMD:C_0603_1608Metric, symbol Device:C
- added C_USB0_OUT_BULK, C_USB1_OUT_BULK: 47uF, Capacitor_SMD:C_1210_3225Metric, symbol Device:C
- added C_USB0_OUT_OPT, C_USB1_OUT_OPT: 100uF DNP, Capacitor_SMD:C_1210_3225Metric, symbol Device:C
- added C_USB_PWR_LOCAL: 10uF, Capacitor_SMD:C_0805_2012Metric, symbol Device:C
- added R_USB0_SHUNT, R_USB1_SHUNT: 0R / SHUNT OPTION, Resistor_SMD:R_1206_3216Metric, symbol Device:R_US
- added R_U_USB0_EN_PD, R_U_USB1_EN_PD: 100k, Resistor_SMD:R_0603_1608Metric, symbol Device:R_US
- added R_U_USB0_FLT_PU, R_U_USB1_FLT_PU: 10k, Resistor_SMD:R_0603_1608Metric, symbol Device:R_US
- added R_U_USB0_ILIM: 54.9k 1%, Resistor_SMD:R_0603_1608Metric, symbol Device:R_US
- added R_U_USB1_ILIM: 34.8k 1%, Resistor_SMD:R_0603_1608Metric, symbol Device:R_US
- added U_USB0, U_USB1: TPS25221DRVR, Package_SON:WSON-6-1EP_2x2mm_P0.65mm_EP1x1.6mm, symbol Pajoniiir-M1:TPS25221DRV
Connections:
- new net 3V3_SYS: R_U_USB0_FLT_PU.1, R_U_USB1_FLT_PU.1
- new net 5V_SYS: C_USB0_IN.1, C_USB1_IN.1, C_USB_PWR_LOCAL.1
- new net GND: C_USB0_IN.2, C_USB0_OUT_BULK.2, C_USB0_OUT_HF.2, C_USB0_OUT_OPT.2, C_USB1_IN.2, C_USB1_OUT_BULK.2, C_USB1_OUT_HF.2, C_USB1_OUT_OPT.2, C_USB_PWR_LOCAL.2, R_U_USB0_EN_PD.1, R_U_USB0_ILIM.2, R_U_USB1_EN_PD.1, R_U_USB1_ILIM.2
- new net USB0_FAULT_N: R_U_USB0_FLT_PU.2
- new net USB0_PWR_EN: R_U_USB0_EN_PD.2
- new net USB0_SW_OUT: R_USB0_SHUNT.1
- new net USB0_VBUS: C_USB0_OUT_BULK.1, C_USB0_OUT_HF.1, C_USB0_OUT_OPT.1, R_USB0_SHUNT.2
- new net USB1_FAULT_N: R_U_USB1_FLT_PU.2
- new net USB1_PWR_EN: R_U_USB1_EN_PD.2
- new net USB1_SW_OUT: R_USB1_SHUNT.1
- new net USB1_VBUS: C_USB1_OUT_BULK.1, C_USB1_OUT_HF.1, C_USB1_OUT_OPT.1, R_USB1_SHUNT.2
Other:
- note added: "Both ports default OFF with 100k EN pulldowns. FAULT is active-low open-drain with 10k pull-up to 3V3_SYS."
- note added: "DRV/WSON pin map: 1 OUT, 2 ILIM, 3 FAULT, 4 EN, 5 GND, 6 IN, exposed pad 7 GND."
- note added: "Per-port output: 100nF + 47uF initial + 100uF DNP tuning. Route with USB_VBUS_HIGH_CURRENT class."
- note added: "USB0: RILIM 54.9k (~1.0A nominal initial). USB1: RILIM 34.8k (~1.6A nominal initial). Final values require EVT characterization."
