File: hardware/Pajoniiir-M1/06_USB_POWER.kicad_sch (KiCad schematic)
At the start: 19 parts

Commit message: hardware: normalize schematic reference designators
Parts:
- renumbered C_USB_PWR_LOCAL to C68, C_USB0_IN to C69, C_USB0_OUT_HF to C70, C_USB0_OUT_BULK to C71, C_USB0_OUT_OPT to C72, C_USB1_IN to C73, C_USB1_OUT_HF to C74, C_USB1_OUT_BULK to C75, C_USB1_OUT_OPT to C76, R_U_USB0_EN_PD to R59, R_U_USB0_FLT_PU to R60, R_U_USB0_ILIM to R61, R_USB0_SHUNT to R62, R_U_USB1_EN_PD to R63, R_U_USB1_FLT_PU to R64, R_U_USB1_ILIM to R65, R_USB1_SHUNT to R66, U_USB1 to U12, U_USB0 to U6
