File: hardware/Pajoniiir-M1/15_DNP_OPTIONS.kicad_sch (KiCad schematic)
At the start: 0 parts

Commit message: hardware: define Rev A assembly option matrix
Other:
- note added: "01: input bulk alternatives = DNP tuning; 02: FB_C6 / FB_AUDIO are 0R defaults with ferrite option; 10: FB_LCD; 11: FB_TOUCH."
- note added: "1. Authoritative LCD panel MPN + FPC pin order + pitch/contact-side + 30-vs-32 resolution."
- note added: "10: DSI six inline 0R = POP. R_LCD_TE_SER = DNP. No external MIPI ESD baseline. Physical J_LCD footprint remains BLOCKED, not DNP."
- note added: "11: R_TOUCH_SDA_PU2 / R_TOUCH_SCL_PU2 = DNP pull-up tuning. Optional touch ESD remains uninstantiated until enclosure exposure requires it."
- note added: "14: INA238 is POP for EVT/DVT and may become DNP in production. R_SYS_SHUNT must remain populated or be replaced by approved footprint-compatible 0R jumper."
- note added: "2. Exact USB-A mechanical connector MPNs / board-edge placement."
- note added: "3. Exact microSD socket MPN / card-detect mechanics."
- note added: "4. RCA / optional 3.5mm mechanical MPNs and enclosure datum."
- note added: "5. PCB fab stackup for 90R USB and 100R MIPI controlled impedance."
- note added: "6. Final high-current shunt / inductor package choices after placement and thermal review."
- note added: "ASSEMBLY POLICY"
- note added: "AUDIO"
- note added: "C_SD_OUT_OPT = 22uF DNP. C_SD_CLK_TUNE = DNP SI tuning. Optional low-C SD ESD waits for final socket/layout. TPS22918 is mandatory POP."
- note added: "DEBUG / FACTORY"
- note added: "DISPLAY / TOUCH"
- note added: "DVT: retain telemetry and selected tuning values; validate EMI/SI/thermal margins and decide cost-down."
- note added: "EVT: populate INA238; expose all tuning/test infrastructure; debug fixtures remain DNL pads."
- note added: "FLASH / CLOCK"
- note added: "Functional DNP/tuning footprints live on their owning sheets. This sheet is control documentation only."
- note added: "HARD GATES BEFORE PCB FREEZE"
- note added: "JDBG_P4 and JDBG_C6 = DNL Tag-Connect PCB pads. JDBG_USB = DNL pogo footprint. C_P4_USBJTAG_DM/DP = DNP tuning."
- note added: "J_LINE_35 = DNP optional line-level output. No headphone amp, speaker amp, ES8311, microphone or legacy monitor-I2S DNP footprints."
- note added: "MICROSD"
- note added: "NO ES8311"
- note added: "NO ESP32-S3"
- note added: "NO MAX485 / RS485"
- note added: "NO MIPI CSI camera block"
- note added: "NO P4<->S3 legacy UART bridge"
- note added: "NO analog microphone"
- note added: "NO battery charger / IP5306 baseline"
- note added: "NO generic large expansion header"
- note added: "NO legacy monitor I2S bridge"
- note added: "NO speaker amplifier / speaker connector"
- note added: "POWER"
- note added: "PROD: only validated tuning values; optional telemetry decision after DVT; no open main power path allowed."
- note added: "PROHIBITED LEGACY FOOTPRINTS"
- note added: "QSPI series 0R tuning footprints POP. Crystal load values are assembly-selection values, not simultaneously populated alternatives."
- note added: "RULE: if a DNP footprint has no named EVT/DVT test or future function, remove it before layout."
- note added: "R_USB0_DM/DP = 0R POP tuning. C_USB0_OUT_OPT = 100uF DNP. Shield 1nF + 1M options DNP. No CMC in Rev A baseline."
- note added: "R_USB1_DM/DP = 22R POP initial. C_USB1_DM/DP = DNP EMI tuning. C_USB1_OUT_OPT = 100uF DNP. Shield 1nF + 1M options DNP."
- note added: "USB0 HIGH-SPEED"
- note added: "USB1 FULL-SPEED"
- note added: "VARIANT INTENT"
Changed lines of the file:
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@@
   (generator "eeschema")
   (generator_version "9.0")
-  (paper "A4")
+  (paper "A3")
   (title_block
     (title "Pajoniiir-M1 Rev A — 15_DNP_OPTIONS")
@@
     (rev "A / M1-SCH-A")
     (company "Pajoniiir")
-    (comment 1 "BOM authority: docs/Pajoniiir_Mainboard_BOM_v0.2.md")
-    (comment 2 "GPIO authority: docs/Pajoniiir_Global_GPIO_Allocation_v0.1.md")
+    (comment 1 "Assembly variant / DNP / DNL authority")
+    (comment 2 "No functional circuitry is duplicated on this sheet")
   )
+  (text "ASSEMBLY POLICY" (exclude_from_sim no) (at 35 25 0) (effects (font (size 1.8 1.8))))
+  (text "Functional DNP/tuning footprints live on their owning sheets. This sheet is control documentation only." (exclude_from_sim no) (at 35 31 0) (effects (font (size 1.27 1.27))))
+  (text "POWER" (exclude_from_sim no) (at 35 42 0) (effects (font (size 1.5 1.5))))
+  (text "01: input bulk alternatives = DNP tuning; 02: FB_C6 / FB_AUDIO are 0R defaults with ferrite option; 10: FB_LCD; 11: FB_TOUCH." (exclude_from_sim no) (at 35 47 0) (effects (font (size 1.27 1.27))))
+  (text "14: INA238 is POP for EVT/DVT and may become DNP in production. R_SYS_SHUNT must remain populated or be replaced by approved footprint-compatible 0R jumper." (exclude_from_sim no) (at 35 52 0) (effects (font (size 1.27 1.27))))
+  (text "USB0 HIGH-SPEED" (exclude_from_sim no) (at 35 64 0) (effects (font (size 1.5 1.5))))
+  (text "R_USB0_DM/DP = 0R POP tuning. C_USB0_OUT_OPT = 100uF DNP. Shield 1nF + 1M options DNP. No CMC in Rev A baseline." (exclude_from_sim no) (at 35 69 0) (effects (font (size 1.27 1.27))))
+  (text "USB1 FULL-SPEED" (exclude_from_sim no) (at 35 81 0) (effects (font (size 1.5 1.5))))
+  (text "R_USB1_DM/DP = 22R POP initial. C_USB1_DM/DP = DNP EMI tuning. C_USB1_OUT_OPT = 100uF DNP. Shield 1nF + 1M options DNP." (exclude_from_sim no) (at 35 86 0) (effects (font (size 1.27 1.27))))
+  (text "FLASH / CLOCK" (exclude_from_sim no) (at 35 98 0) (effects (font (size 1.5 1.5))))
+  (text "QSPI series 0R tuning footprints POP. Crystal load values are assembly-selection values, not simultaneously populated alternatives." (exclude_from_sim no) (at 35 103 0) (effects (font (size 1.27 1.27))))
+  (text "AUDIO" (exclude_from_sim no) (at 35 115 0) (effects (font (size 1.5 1.5))))
+  (text "J_LINE_35 = DNP optional line-level output. No headphone amp, speaker amp, ES8311, microphone or legacy monitor-I2S DNP footprints." (exclude_from_sim no) (at 35 120 0) (effects (font (size 1.27 1.27))))
+  (text "DISPLAY / TOUCH" (exclude_from_sim no) (at 35 132 0) (effects (font (size 1.5 1.5))))
+  (text "10: DSI six inline 0R = POP. R_LCD_TE_SER = DNP. No external MIPI ESD baseline. Physical J_LCD footprint remains BLOCKED, not DNP." (exclude_from_sim no) (at 35 137 0) (effects (font (size 1.27 1.27))))
+  (text "11: R_TOUCH_SDA_PU2 / R_TOUCH_SCL_PU2 = DNP pull-up tuning. Optional touch ESD remains uninstantiated until enclosure exposure requires it." (exclude_from_sim no) (at 35 142 0) (effects (font (size 1.27 1.27))))
+  (text "MICROSD" (exclude_from_sim no) (at 35 154 0) (effects (font (size 1.5 1.5))))
+  (text "C_SD_OUT_OPT = 22uF DNP. C_SD_CLK_TUNE = DNP SI tuning. Optional low-C SD ESD waits for final socket/layout. TPS22918 is mandatory POP." (exclude_from_sim no) (at 35 159 0) (effects (font (size 1.27 1.27))))
+  (text "DEBUG / FACTORY" (exclude_from_sim no) (at 35 171 0) (effects (font (size 1.5 1.5))))
+  (text "JDBG_P4 and JDBG_C6 = DNL Tag-Connect PCB pads. JDBG_USB = DNL pogo footprint. C_P4_USBJTAG_DM/DP = DNP tuning." (exclude_from_sim no) (at 35 176 0) (effects (font (size 1.27 1.27))))
+  (text "PROHIBITED LEGACY FOOTPRINTS" (exclude_from_sim no) (at 170 42 0) (effects (font (size 1.5 1.5))))
+  (text "NO ESP32-S3" (exclude_from_sim no) (at 170 48 0) (effects (font (size 1.27 1.27))))
+  (text "NO ES8311" (exclude_from_sim no) (at 170 53 0) (effects (font (size 1.27 1.27))))
+  (text "NO speaker amplifier / speaker connector" (exclude_from_sim no) (at 170 58 0) (effects (font (size 1.27 1.27))))
+  (text "NO analog microphone" (exclude_from_sim no) (at 170 63 0) (effects (font (size 1.27 1.27))))
+  (text "NO MAX485 / RS485" (exclude_from_sim no) (at 170 68 0) (effects (font (size 1.27 1.27))))
+  (text "NO MIPI CSI camera block" (exclude_from_sim no) (at 170 73 0) (effects (font (size 1.27 1.27))))
+  (text "NO P4<->S3 legacy UART bridge" (exclude_from_sim no) (at 170 78 0) (effects (font (size 1.27 1.27))))
+  (text "NO legacy monitor I2S bridge" (exclude_from_sim no) (at 170 83 0) (effects (font (size 1.27 1.27))))
+  (text "NO battery charger / IP5306 baseline" (exclude_from_sim no) (at 170 88 0) (effects (font (size 1.27 1.27))))
+  (text "NO generic large expansion header" (exclude_from_sim no) (at 170 93 0) (effects (font (size 1.27 1.27))))
+  (text "VARIANT INTENT" (exclude_from_sim no) (at 170 108 0) (effects (font (size 1.5 1.5))))
+  (text "EVT: populate INA238; expose all tuning/test infrastructure; debug fixtures remain DNL pads." (exclude_from_sim no) (at 170 114 0) (effects (font (size 1.27 1.27))))
+  (text "DVT: retain telemetry and selected tuning values; validate EMI/SI/thermal margins and decide cost-down." (exclude_from_sim no) (at 170 119 0) (effects (font (size 1.27 1.27))))
+  (text "PROD: only validated tuning values; optional telemetry decision after DVT; no open main power path allowed." (exclude_from_sim no) (at 170 124 0) (effects (font (size 1.27 1.27))))
+  (text "HARD GATES BEFORE PCB FREEZE" (exclude_from_sim no) (at 170 139 0) (effects (font (size 1.5 1.5))))
+  (text "1. Authoritative LCD panel MPN + FPC pin order + pitch/contact-side + 30-vs-32 resolution." (exclude_from_sim no) (at 170 145 0) (effects (font (size 1.27 1.27))))
+  (text "2. Exact USB-A mechanical connector MPNs / board-edge placement." (exclude_from_sim no) (at 170 150 0) (effects (font (size 1.27 1.27))))
+  (text "3. Exact microSD socket MPN / card-detect mechanics." (exclude_from_sim no) (at 170 155 0) (effects (font (size 1.27 1.27))))
+  (text "4. RCA / optional 3.5mm mechanical MPNs and enclosure datum." (exclude_from_sim no) (at 170 160 0) (effects (font (size 1.27 1.27))))
+  (text "5. PCB fab stackup for 90R USB and 100R MIPI controlled impedance." (exclude_from_sim no) (at 170 165 0) (effects (font (size 1.27 1.27))))
+  (text "6. Final high-current shunt / inductor package choices after placement and thermal review." (exclude_from_sim no) (at 170 170 0) (effects (font (size 1.27 1.27))))
+  (text "RULE: if a DNP footprint has no named EVT/DVT test or future function, remove it before layout." (exclude_from_sim no) (at 170 183 0) (effects (font (size 1.35 1.35))))
   (sheet_instances
     (path "/" (page "16"))
