File: hardware/Pajoniiir-M1/14_TEST_MONITORING.kicad_sch (KiCad schematic)
At the start: 0 parts

Commit message: hardware: capture total-system power monitoring schematic
Parts:
- added C_INA_DIFF, C_INA_HF: 100nF, Capacitor_SMD:C_0603_1608Metric, symbol Device:C
- added C_INA_LOCAL: 1uF, Capacitor_SMD:C_0603_1608Metric, symbol Device:C
- added R_INA_ALERT_PU: 10k, Resistor_SMD:R_0603_1608Metric, symbol Device:R_US
- added R_INA_N, R_INA_P: 10R, Resistor_SMD:R_0603_1608Metric, symbol Device:R_US
- added R_SYS_SHUNT: 5mR 1% >=1W KELVIN, symbol Device:R_US
- added TP_3V3_SYS: 3V3_SYS, TestPoint:TestPoint_Pad_D1.5mm, symbol Connector:TestPoint
- added TP_5V_PROTECTED: 5V_PROTECTED, TestPoint:TestPoint_Pad_D1.5mm, symbol Connector:TestPoint
- added TP_5V_SYS: 5V_SYS, TestPoint:TestPoint_Pad_D1.5mm, symbol Connector:TestPoint
- added TP_SYS_ALERT: SYS_POWER_ALERT_N, TestPoint:TestPoint_Pad_D1.5mm, symbol Connector:TestPoint
- added U_MON: INA238AIDGSR, Package_SO:VSSOP-10_3x3mm_P0.5mm, symbol Pajoniiir-M1:INA238
Connections:
- new net 3V3_SYS: C_INA_HF.1, C_INA_LOCAL.1, R_INA_ALERT_PU.1, TP_3V3_SYS.1
- new net 5V_PROTECTED: R_INA_P.1, R_SYS_SHUNT.1, TP_5V_PROTECTED.1
- new net 5V_SYS: R_INA_N.1, R_SYS_SHUNT.2, TP_5V_SYS.1
- new net GND: C_INA_HF.2, C_INA_LOCAL.2
- new net INA_INN_FILT: C_INA_DIFF.2
- new net INA_INP_FILT: C_INA_DIFF.1, R_INA_P.2
- new net SYS_POWER_ALERT_N: R_INA_ALERT_PU.2, TP_SYS_ALERT.1
Other:
- note added: "Cost-down: U_MON/filter/ALERT may be DNP, but R_SYS_SHUNT must remain or be replaced by footprint-compatible 0R high-current jumper."
- note added: "INA238 address 0x40: A0=A1=GND. VBUS senses load-side 5V_SYS; IN+ = supply-side Kelvin, IN- = load-side Kelvin."
- note added: "Input filter: 10R + 10R and 100nF differential. Do not route sense traces on shared high-current copper; take Kelvin taps at shunt pads."
- note added: "R_SYS_SHUNT = 5mR 1%, >=1W; use true Kelvin/4-terminal footprint if available. At 4.5A: 22.5mV, ~101mW."
- note added: "Shared I2C uses existing bus pull-ups; do not add another strong pull-up pair on this sheet."

Commit message: hardware: lock Kelvin system shunt candidate
Parts:
- R_SYS_SHUNT: value 5mR 1% >=1W KELVIN -> WSK25125L000FEA / 5mR 1% 1W; footprint (none) -> Resistor_SMD:R_Shunt_Vishay_WSK2512_6332Metric_T1.19mm
Other:
- note added: "R_SYS_SHUNT = WSK25125L000FEA, 5mR 1% 1W, 4-terminal/Kelvin. At 4.5A: 22.5mV, ~101mW."
- note removed: "R_SYS_SHUNT = 5mR 1%, >=1W; use true Kelvin/4-terminal footprint if available. At 4.5A: 22.5mV, ~101mW."
Changed lines of the file:
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@@
     (exclude_from_sim no) (in_bom yes) (on_board yes) (dnp no)
     (property "Reference" "R_SYS_SHUNT" (at 88 43 0) (effects (font (size 1.27 1.27))))
-    (property "Value" "5mR 1% >=1W KELVIN" (at 88 47 0) (effects (font (size 1.27 1.27))))
-    (property "Footprint" "" (at 85 45 0) (effects (font (size 1.27 1.27)) (hide yes)))
-    (property "Datasheet" "~" (at 85 45 0) (effects (font (size 1.27 1.27)) (hide yes)))
+    (property "Value" "WSK25125L000FEA / 5mR 1% 1W" (at 88 47 0) (effects (font (size 1.27 1.27))))
+    (property "Footprint" "Resistor_SMD:R_Shunt_Vishay_WSK2512_6332Metric_T1.19mm" (at 85 45 0) (effects (font (size 1.27 1.27)) (hide yes)))
+    (property "Datasheet" "https://www.vishay.com/docs/30108/wsk2512.pdf" (at 85 45 0) (effects (font (size 1.27 1.27)) (hide yes)))
     (pin "1") (pin "2")
     (instances (project "Pajoniiir-M1" (path "/2c8dd352-b7b8-4d9e-8f93-5dd43be2a100/3100000e-6b2a-4a3a-8c91-00000000000e" (reference "R_SYS_SHUNT") (unit 1))))
@@
   )
   (label "SYS_POWER_ALERT_N" (at 130 105 0) (effects (font (size 1.27 1.27))))
-  (text "R_SYS_SHUNT = 5mR 1%, >=1W; use true Kelvin/4-terminal footprint if available. At 4.5A: 22.5mV, ~101mW." (exclude_from_sim no) (at 35 125 0) (effects (font (size 1.27 1.27))))
+  (text "R_SYS_SHUNT = WSK25125L000FEA, 5mR 1% 1W, 4-terminal/Kelvin. At 4.5A: 22.5mV, ~101mW." (exclude_from_sim no) (at 35 125 0) (effects (font (size 1.27 1.27))))
   (text "INA238 address 0x40: A0=A1=GND. VBUS senses load-side 5V_SYS; IN+ = supply-side Kelvin, IN- = load-side Kelvin." (exclude_from_sim no) (at 35 130 0) (effects (font (size 1.27 1.27))))
   (text "Input filter: 10R + 10R and 100nF differential. Do not route sense traces on shared high-current copper; take Kelvin taps at shunt pads." (exclude_from_sim no) (at 35 135 0) (effects (font (size 1.27 1.27))))
