File: hardware/Pajoniiir-M1/14_TEST_MONITORING.kicad_sch (KiCad schematic)
At the start: 12 parts, among them U14 INA238AIDGSR

Commit message: display: migrate schematic to final DSI506 module
Connections:
- net I2C_SCL renamed DISPLAY_I2C_SCL
- net I2C_SDA renamed DISPLAY_I2C_SDA
Changed lines of the file:
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@@
     (instances (project "Pajoniiir-M1" (path "/2c8dd352-b7b8-4d9e-8f93-5dd43be2a100/3100000e-6b2a-4a3a-8c91-00000000000e" (reference "#PWR1405") (unit 1))))
   )
-  (hierarchical_label "I2C_SDA" (shape bidirectional) (at 215.265 74.93 0) (effects (font (size 1.27 1.27))))
+  (hierarchical_label "DISPLAY_I2C_SDA" (shape bidirectional) (at 215.265 74.93 0) (effects (font (size 1.27 1.27))))
   (wire (pts (xy 175.26 74.93) (xy 215.265 74.93)) (stroke (width 0) (type default)))
-  (hierarchical_label "I2C_SCL" (shape input) (at 215.265 77.47 0) (effects (font (size 1.27 1.27))))
+  (hierarchical_label "DISPLAY_I2C_SCL" (shape input) (at 215.265 77.47 0) (effects (font (size 1.27 1.27))))
   (wire (pts (xy 175.26 77.47) (xy 215.265 77.47)) (stroke (width 0) (type default)))
   (hierarchical_label "SYS_POWER_ALERT_N" (shape output) (at 175.26 82.55 0) (effects (font (size 1.27 1.27))))

Commit message: feat: establish board-first B8 pre-layout
Populate the live PCB with the complete schematic footprint/net set, preserve fail-closed mechanical gates, and isolate DSI506 as a qualified display profile. Add reproducible placement validation, ERC/BOM evidence, and synchronized project documentation.
Parts:
- U14: footprint Package_SO:VSSOP-10_3x3mm_P0.5mm -> Pajoniiir-M1:Texas_DGS0010A_VSSOP-10_3x3mm_P0.5mm
Changed lines of the file:
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@@
     (property "Reference" "U14" (at 154.1 55.93 0) (effects (font (size 1.27 1.27))))
     (property "Value" "INA238AIDGSR" (at 154.1 58.93 0) (effects (font (size 1.27 1.27))))
-    (property "Footprint" "Package_SO:VSSOP-10_3x3mm_P0.5mm" (at 165.1 74.93 0) (effects (font (size 1.27 1.27)) (hide yes)))
+    (property "Footprint" "Pajoniiir-M1:Texas_DGS0010A_VSSOP-10_3x3mm_P0.5mm" (at 165.1 74.93 0) (effects (font (size 1.27 1.27)) (hide yes)))
     (property "Datasheet" "https://www.ti.com/lit/ds/symlink/ina238.pdf" (at 165.1 74.93 0) (effects (font (size 1.27 1.27)) (hide yes)))
     (pin "1") (pin "2") (pin "3") (pin "4") (pin "5")
