File: hardware/Pajoniiir-M1/13_DEBUG_SERVICE.kicad_sch (KiCad schematic)
At the start: 15 parts

Commit message: hardware: bind remaining hierarchical ports to nets
Changed lines of the file:
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@@
     (comment 2 "VREF pins are sense-only; fixtures must not back-power board")
   )
-  (hierarchical_label "3V3_SYS" (shape input) (at 24.765 29.845 0) (effects (font (size 1.27 1.27))))
-  (hierarchical_label "DEBUG_UART_TX" (shape input) (at 24.765 34.925 0) (effects (font (size 1.27 1.27))))
-  (hierarchical_label "DEBUG_UART_RX" (shape output) (at 24.765 40.005 0) (effects (font (size 1.27 1.27))))
-  (hierarchical_label "CHIP_PU" (shape bidirectional) (at 24.765 45.085 0) (effects (font (size 1.27 1.27))))
-  (hierarchical_label "BOOT_GPIO35" (shape bidirectional) (at 24.765 50.165 0) (effects (font (size 1.27 1.27))))
-  (hierarchical_label "BOOT_GPIO36" (shape bidirectional) (at 24.765 55.245 0) (effects (font (size 1.27 1.27))))
-  (hierarchical_label "P4_USBJTAG_DM" (shape bidirectional) (at 24.765 59.69 0) (effects (font (size 1.27 1.27))))
-  (hierarchical_label "P4_USBJTAG_DP" (shape bidirectional) (at 24.765 64.77 0) (effects (font (size 1.27 1.27))))
-  (hierarchical_label "3V3_C6" (shape input) (at 24.765 74.93 0) (effects (font (size 1.27 1.27))))
-  (hierarchical_label "C6_UART_TX" (shape input) (at 24.765 80.01 0) (effects (font (size 1.27 1.27))))
-  (hierarchical_label "C6_UART_RX" (shape output) (at 24.765 85.09 0) (effects (font (size 1.27 1.27))))
-  (hierarchical_label "C6_EN" (shape bidirectional) (at 24.765 90.17 0) (effects (font (size 1.27 1.27))))
-  (hierarchical_label "C6_BOOT_GPIO8" (shape bidirectional) (at 24.765 95.25 0) (effects (font (size 1.27 1.27))))
-  (hierarchical_label "C6_BOOT_GPIO9" (shape bidirectional) (at 24.765 99.695 0) (effects (font (size 1.27 1.27))))
+  (hierarchical_label "3V3_SYS" (shape input) (at 85.09 47.625 0) (effects (font (size 1.27 1.27))))
+  (hierarchical_label "DEBUG_UART_TX" (shape input) (at 97.79 47.625 0) (effects (font (size 1.27 1.27))))
+  (hierarchical_label "DEBUG_UART_RX" (shape output) (at 85.09 45.085 0) (effects (font (size 1.27 1.27))))
+  (hierarchical_label "CHIP_PU" (shape bidirectional) (at 97.79 45.085 0) (effects (font (size 1.27 1.27))))
+  (hierarchical_label "BOOT_GPIO35" (shape bidirectional) (at 97.79 42.545 0) (effects (font (size 1.27 1.27))))
+  (hierarchical_label "BOOT_GPIO36" (shape bidirectional) (at 149.86 45.085 0) (effects (font (size 1.27 1.27))))
+  (hierarchical_label "P4_USBJTAG_DM" (shape bidirectional) (at 111.125 64.77 0) (effects (font (size 1.27 1.27))))
+  (hierarchical_label "P4_USBJTAG_DP" (shape bidirectional) (at 111.125 74.93 0) (effects (font (size 1.27 1.27))))
+  (hierarchical_label "3V3_C6" (shape input) (at 85.09 97.79 0) (effects (font (size 1.27 1.27))))
+  (hierarchical_label "C6_UART_TX" (shape input) (at 97.79 97.79 0) (effects (font (size 1.27 1.27))))
+  (hierarchical_label "C6_UART_RX" (shape output) (at 85.09 95.25 0) (effects (font (size 1.27 1.27))))
+  (hierarchical_label "C6_EN" (shape bidirectional) (at 97.79 95.25 0) (effects (font (size 1.27 1.27))))
+  (hierarchical_label "C6_BOOT_GPIO8" (shape bidirectional) (at 149.86 95.25 0) (effects (font (size 1.27 1.27))))
+  (hierarchical_label "C6_BOOT_GPIO9" (shape bidirectional) (at 97.79 92.71 0) (effects (font (size 1.27 1.27))))
   (symbol
     (lib_id "Connector_Generic:Conn_02x03_Odd_Even") (at 90.17 45.085 0) (unit 1)
@@
     (instances (project "Pajoniiir-M1" (path "/2c8dd352-b7b8-4d9e-8f93-5dd43be2a100/3100000d-6b2a-4a3a-8c91-00000000000d" (reference "JDBG_P4") (unit 1))))
   )
-  (label "3V3_SYS" (at 85.09 47.625 0) (effects (font (size 1.27 1.27))))
-  (label "DEBUG_UART_TX" (at 97.79 47.625 0) (effects (font (size 1.27 1.27))))
-  (label "DEBUG_UART_RX" (at 85.09 45.085 0) (effects (font (size 1.27 1.27))))
-  (label "CHIP_PU" (at 97.79 45.085 0) (effects (font (size 1.27 1.27))))
   (symbol
     (lib_id "power:GND") (at 85.09 42.545 0) (unit 1)
@@
     (instances (project "Pajoniiir-M1" (path "/2c8dd352-b7b8-4d9e-8f93-5dd43be2a100/3100000d-6b2a-4a3a-8c91-00000000000d" (reference "#PWR_JDBG_P4_5") (unit 1))))
   )
-  (label "BOOT_GPIO35" (at 97.79 42.545 0) (effects (font (size 1.27 1.27))))
   (symbol
     (lib_id "Device:R_US") (at 114.935 64.77 90) (unit 1)
@@
     (instances (project "Pajoniiir-M1" (path "/2c8dd352-b7b8-4d9e-8f93-5dd43be2a100/3100000d-6b2a-4a3a-8c91-00000000000d" (reference "R_USBJTAG_DM") (unit 1))))
   )
-  (label "P4_USBJTAG_DM" (at 111.125 64.77 0) (effects (font (size 1.27 1.27))))
   (wire (pts (xy 118.745 64.77) (xy 144.78 64.77)) (stroke (width 0) (type default)))
   (label "USBJTAG_DM_SERVICE" (at 130.175 64.77 0) (effects (font (size 1.27 1.27))))
@@
     (instances (project "Pajoniiir-M1" (path "/2c8dd352-b7b8-4d9e-8f93-5dd43be2a100/3100000d-6b2a-4a3a-8c91-00000000000d" (reference "R_USBJTAG_DP") (unit 1))))
   )
-  (label "P4_USBJTAG_DP" (at 111.125 74.93 0) (effects (font (size 1.27 1.27))))
   (wire (pts (xy 118.745 74.93) (xy 144.78 74.93)) (stroke (width 0) (type default)))
   (label "USBJTAG_DP_SERVICE" (at 130.175 74.93 0) (effects (font (size 1.27 1.27))))
@@
     (instances (project "Pajoniiir-M1" (path "/2c8dd352-b7b8-4d9e-8f93-5dd43be2a100/3100000d-6b2a-4a3a-8c91-00000000000d" (reference "JDBG_C6") (unit 1))))
   )
-  (label "3V3_C6" (at 85.09 97.79 0) (effects (font (size 1.27 1.27))))
-  (label "C6_UART_TX" (at 97.79 97.79 0) (effects (font (size 1.27 1.27))))
-  (label "C6_UART_RX" (at 85.09 95.25 0) (effects (font (size 1.27 1.27))))
-  (label "C6_EN" (at 97.79 95.25 0) (effects (font (size 1.27 1.27))))
   (symbol
     (lib_id "power:GND") (at 85.09 92.71 0) (unit 1)
@@
     (instances (project "Pajoniiir-M1" (path "/2c8dd352-b7b8-4d9e-8f93-5dd43be2a100/3100000d-6b2a-4a3a-8c91-00000000000d" (reference "#PWR_JDBG_C6_5") (unit 1))))
   )
-  (label "C6_BOOT_GPIO9" (at 97.79 92.71 0) (effects (font (size 1.27 1.27))))
   (symbol
     (lib_id "Connector:TestPoint") (at 149.86 45.085 0) (unit 1)
@@
     (instances (project "Pajoniiir-M1" (path "/2c8dd352-b7b8-4d9e-8f93-5dd43be2a100/3100000d-6b2a-4a3a-8c91-00000000000d" (reference "TP_P4_BOOT36") (unit 1))))
   )
-  (label "BOOT_GPIO36" (at 149.86 45.085 0) (effects (font (size 1.27 1.27))))
   (symbol
     (lib_id "Connector:TestPoint") (at 149.86 95.25 0) (unit 1)
@@
     (instances (project "Pajoniiir-M1" (path "/2c8dd352-b7b8-4d9e-8f93-5dd43be2a100/3100000d-6b2a-4a3a-8c91-00000000000d" (reference "TP_C6_GPIO8") (unit 1))))
   )
-  (label "C6_BOOT_GPIO8" (at 149.86 95.25 0) (effects (font (size 1.27 1.27))))
   (symbol
     (lib_id "Connector:TestPoint") (at 205.105 34.925 0) (unit 1)
