File: hardware/Pajoniiir-M1/13_DEBUG_SERVICE.kicad_sch (KiCad schematic)
At the start: 15 parts, among them J10 C6 DEBUG TC2030-NL DNL, J8 P4 DEBUG TC2030-NL DNL, J9 P4 USB SERIAL/JTAG POGO DNL

Commit message: mechanical: close J9 factory pogo gate
Parts:
- J9: value P4 USB SERIAL/JTAG POGO DNL -> P4 USB SERIAL/JTAG FACTORY POGO DNL; footprint (none) -> Pajoniiir-M1:Factory_Pogo_USBJTAG_1x05_P1.27_2Tooling
Changed lines of the file:
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@@
     (exclude_from_sim no) (in_bom no) (on_board yes) (dnp yes)
     (property "Reference" "J9" (at 184.785 57.85 0) (effects (font (size 1.27 1.27))))
-    (property "Value" "P4 USB SERIAL/JTAG POGO DNL" (at 184.785 60.35 0) (effects (font (size 1.27 1.27))))
-    (property "Footprint" "" (at 184.785 69.85 0) (effects (font (size 1.27 1.27)) (hide yes)))
+    (property "Value" "P4 USB SERIAL/JTAG FACTORY POGO DNL" (at 184.785 60.35 0) (effects (font (size 1.27 1.27))))
+    (property "Footprint" "Pajoniiir-M1:Factory_Pogo_USBJTAG_1x05_P1.27_2Tooling" (at 184.785 69.85 0) (effects (font (size 1.27 1.27)) (hide yes)))
     (property "Datasheet" "~" (at 184.785 69.85 0) (effects (font (size 1.27 1.27)) (hide yes)))
     (pin "1") (pin "2") (pin "3") (pin "4") (pin "5")
