File: hardware/Pajoniiir-M1/05_C6_WIFI.kicad_sch (KiCad schematic)
At the start: 22 parts, among them U4 ESP32-C6-WROOM-1-N4

Commit message: hardware: correct C6 power and interface pin mapping
Connections:
- net 3V3_C6: now also U4.2 (3V3); no longer R_SDIO_D0.1, R_SDIO_D0.2, R_SDIO_D0_PU.2, R_SDIO_D1.1, R_SDIO_D1.2, R_SDIO_D1_PU.2, R_SDIO_D2.1, R_SDIO_D2.2, R_SDIO_D2_PU.2, R_SDIO_D3.1, R_SDIO_D3.2, R_SDIO_D3_PU.2, U4.1 (GND), U4.13 (GPIO12/USB_D-), U4.28 (GND), U4.29 (GND)
- net C6_BOOT_GPIO8: now also U4.10 (GPIO8); no longer U4.17 (GPIO19)
- net C6_BOOT_GPIO9: now also U4.15 (GPIO9); no longer U4.16 (GPIO18)
- net C6_EN: now also U4.3 (EN/CHIP_PU)
- net C6_SDIO_CMD: no longer R_SDIO_CMD.1, R_SDIO_CMD_PU.2, U4.15 (GPIO9)
- net GND: now also U4.1 (GND), U4.28 (GND), U4.29 (GND); no longer U4.2 (3V3)
- net C6_SDIO_CLK_C6: now reaches R_SDIO_CLK.1
- net C6_SDIO_CLK_C6: now also U4.17 (GPIO19); no longer U4.10 (GPIO8)
- net C6_SDIO_D0_C6: now reaches U4.18 (GPIO20)
- net C6_SDIO_D0_C6: now also R_SDIO_D0.1, R_SDIO_D0_PU.2
- net C6_SDIO_D1_C6: now reaches U4.19 (GPIO21)
- net C6_SDIO_D1_C6: now also R_SDIO_D1.1, R_SDIO_D1_PU.2
- net C6_SDIO_D2_C6: now reaches U4.20 (GPIO22)
- net C6_SDIO_D2_C6: now also R_SDIO_D2.1, R_SDIO_D2_PU.2
- net C6_SDIO_D3_C6: now reaches U4.21 (GPIO23)
- net C6_SDIO_D3_C6: now also R_SDIO_D3.1, R_SDIO_D3_PU.2
- net at U4.24 (U0RXD/GPIO17): now also R_C6_UART_RX.1
- net at U4.25 (U0TXD/GPIO16): now also R_C6_UART_TX.1
- new net C6_SDIO_CMD_C6: R_SDIO_CMD.1, R_SDIO_CMD_PU.2, U4.16 (GPIO18)
- new net C6_SDIO_D0: R_SDIO_D0.2
- new net C6_SDIO_D1: R_SDIO_D1.2
- new net C6_SDIO_D2: R_SDIO_D2.2
- new net C6_SDIO_D3: R_SDIO_D3.2
Other:
- moved on the sheet: R_C6_UART_RX, R_C6_UART_TX, R_SDIO_CLK, R_SDIO_CMD, R_SDIO_D0, R_SDIO_D1, R_SDIO_D2, R_SDIO_D3

Commit message: hardware: declare verified rail power sources for ERC
Changed lines of the file:
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@@
   (text "C6 recovery remains independent of P4: UART0 TX/RX + GPIO8/GPIO9 + EN are exported to service/debug sheet." (exclude_from_sim no) (at 35 142 0) (effects (font (size 1.27 1.27))))
   (text "RF: place module antenna at PCB edge; preserve official footprint keep-out on every copper layer. If enclosure blocks antenna, switch to WROOM-1U before PCB freeze." (exclude_from_sim no) (at 35 147 0) (effects (font (size 1.27 1.27))))
+  (symbol
+    (lib_id "power:PWR_FLAG")
+    (at 130.175 46.99 0)
+    (unit 1)
+    (exclude_from_sim no)
+    (in_bom yes)
+    (on_board yes)
+    (dnp no)
+    (property "Reference" "#FLG0501" (at 130.175 48.895 0) (effects (font (size 1.27 1.27)) (hide yes)))
+    (property "Value" "PWR_FLAG" (at 130.175 50.800000000000004 0) (effects (font (size 1.27 1.27))))
+    (property "Footprint" "" (at 130.175 46.99 0) (effects (font (size 1.27 1.27)) (hide yes)))
+    (property "Datasheet" "~" (at 130.175 46.99 0) (effects (font (size 1.27 1.27)) (hide yes)))
+    (property "Description" "Special symbol for telling ERC where power comes from" (at 130.175 46.99 0) (effects (font (size 1.27 1.27)) (hide yes)))
+    (pin "1")
+    (instances (project "Pajoniiir-M1" (path "/2c8dd352-b7b8-4d9e-8f93-5dd43be2a100/31000005-6b2a-4a3a-8c91-000000000005" (reference "#FLG0501") (unit 1))))
+  )
   (sheet_instances (path "/" (page "6")))
   (embedded_fonts no)
