File: hardware/Pajoniiir-M1/04_P4_FLASH_CLOCK_RESET.kicad_sch (KiCad schematic)
At the start: 21 parts, among them U2 W25Q128JVPIQ, Y1 ECS-400-10-37B2-CKY-TR

Commit message: ci: capture KiCad 9 symbols and repair PGTH junction
Parts:
- Y1: symbol Pajoniiir-M1:Crystal_GND24_M1 -> Device:Crystal_GND24
Changed lines of the file:
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@@
   )
   (symbol
-    (lib_id "Pajoniiir-M1:Crystal_GND24_M1") (at 189.865 64.77 0) (unit 1)
+    (lib_id "Device:Crystal_GND24") (at 189.865 64.77 0) (unit 1)
     (exclude_from_sim no) (in_bom yes) (on_board yes) (dnp no)
     (property "Reference" "Y1" (at 187.865 56.77 0) (effects (font (size 1.27 1.27))))

Commit message: hardware: pin Rev-A symbols to local library copies
Parts:
- Y1: symbol Device:Crystal_GND24 -> Pajoniiir-M1:Crystal_GND24_M1
Changed lines of the file:
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@@
   )
   (symbol
-    (lib_id "Device:Crystal_GND24") (at 189.865 64.77 0) (unit 1)
+    (lib_id "Pajoniiir-M1:Crystal_GND24_M1") (at 189.865 64.77 0) (unit 1)
     (exclude_from_sim no) (in_bom yes) (on_board yes) (dnp no)
     (property "Reference" "Y1" (at 187.865 56.77 0) (effects (font (size 1.27 1.27))))
