File: hardware/Pajoniiir-M1/02_POWER_3V3.kicad_sch (KiCad schematic)
At the start: 14 parts, among them U8 TPS62132RGTR

Commit message: hardware: stabilize system buck and crystal symbols
Parts:
- U8: symbol Regulator_Switching:TPS62132 -> Pajoniiir-M1:TPS62132_M1
Changed lines of the file:
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@@
   )
   (symbol
-    (lib_id "Regulator_Switching:TPS62132")
+    (lib_id "Pajoniiir-M1:TPS62132_M1")
     (at 120.015 55.245 0) (unit 1)
     (exclude_from_sim no) (in_bom yes) (on_board yes) (dnp no)
