File: hardware/Pajoniiir-M1/02_POWER_3V3.kicad_sch (KiCad schematic)
At the start: 14 parts, among them U8 TPS62132RGTR

Commit message: feat: establish board-first B8 pre-layout
Populate the live PCB with the complete schematic footprint/net set, preserve fail-closed mechanical gates, and isolate DSI506 as a qualified display profile. Add reproducible placement validation, ERC/BOM evidence, and synchronized project documentation.
Parts:
- added TP26: 3V3_PG, TestPoint:TestPoint_Pad_D1.5mm, symbol Connector:TestPoint
Connections:
- net 3V3_PG: now also TP26.1
Changed lines of the file:
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@@
   (sheet_instances (path "/" (page "3")))
   (embedded_fonts no)
+  (symbol (lib_id "Connector:TestPoint") (at 225.425 110.49 0) (unit 1)
+    (exclude_from_sim no) (in_bom yes) (on_board yes) (dnp no)
+    (property "Reference" "TP26" (at 225.425 103.49 0) (effects (font (size 1.27 1.27))))
+    (property "Value" "3V3_PG" (at 225.425 105.49 0) (effects (font (size 1.27 1.27))))
+    (property "Footprint" "TestPoint:TestPoint_Pad_D1.5mm" (at 225.425 110.49 0) (effects (font (size 1.27 1.27)) (hide yes)))
+    (property "Datasheet" "~" (at 225.425 110.49 0) (effects (font (size 1.27 1.27)) (hide yes)))
+    (pin "1")
+    (instances (project "Pajoniiir-M1" (path "/2c8dd352-b7b8-4d9e-8f93-5dd43be2a100/31000002-6b2a-4a3a-8c91-000000000002" (reference "TP26") (unit 1))))
+  )
+  (label "3V3_PG" (at 225.425 110.49 0) (effects (font (size 1.27 1.27))))
 )

Commit message: pcb: fix U8 thermal via drill rule
Parts:
- U8: footprint Package_DFN_QFN:VQFN-16-1EP_3x3mm_P0.5mm_EP1.68x1.68mm_ThermalVias -> Pajoniiir-M1:VQFN-16-1EP_3x3mm_P0.5mm_EP1.68x1.68mm_ThermalVias
Changed lines of the file:
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@@
     (property "Reference" "U8" (at 122.015 38.245 0) (effects (font (size 1.27 1.27))))
     (property "Value" "TPS62132RGTR" (at 122.015 41.245 0) (effects (font (size 1.27 1.27))))
-    (property "Footprint" "Package_DFN_QFN:VQFN-16-1EP_3x3mm_P0.5mm_EP1.68x1.68mm_ThermalVias" (at 120.015 55.245 0) (effects (font (size 1.27 1.27)) (hide yes)))
+    (property "Footprint" "Pajoniiir-M1:VQFN-16-1EP_3x3mm_P0.5mm_EP1.68x1.68mm_ThermalVias" (at 120.015 55.245 0) (effects (font (size 1.27 1.27)) (hide yes)))
     (property "Datasheet" "https://www.ti.com/lit/ds/symlink/tps62130.pdf" (at 120.015 55.245 0) (effects (font (size 1.27 1.27)) (hide yes)))
     (pin "1")
