File: hardware/Pajoniiir-M1/08_USB1_FLX4.kicad_sch (KiCad schematic)
At the start: 9 parts, among them J3 USB-A FLX4 TBD-MECH

Commit message: mechanical: lock USB and RCA footprints
Parts:
- J3: value USB-A FLX4 TBD-MECH -> 87520-1010ALF; footprint (none) -> Pajoniiir-M1:Amphenol_87520-1010ALF
Changed lines of the file:
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@@
     (exclude_from_sim no) (in_bom yes) (on_board yes) (dnp no)
     (property "Reference" "J3" (at 176.785 42.69 0) (effects (font (size 1.27 1.27))))
-    (property "Value" "USB-A FLX4 TBD-MECH" (at 176.785 45.69 0) (effects (font (size 1.27 1.27))))
-    (property "Footprint" "" (at 184.785 59.69 0) (effects (font (size 1.27 1.27)) (hide yes)))
-    (property "Datasheet" "~" (at 184.785 59.69 0) (effects (font (size 1.27 1.27)) (hide yes)))
+    (property "Value" "87520-1010ALF" (at 176.785 45.69 0) (effects (font (size 1.27 1.27))))
+    (property "Footprint" "Pajoniiir-M1:Amphenol_87520-1010ALF" (at 184.785 59.69 0) (effects (font (size 1.27 1.27)) (hide yes)))
+    (property "Datasheet" "https://cdn.amphenol-cs.com/media/wysiwyg/files/drawing/87520.pdf" (at 184.785 59.69 0) (effects (font (size 1.27 1.27)) (hide yes)))
     (pin "1") (pin "2") (pin "3") (pin "4") (pin "5")
     (instances (project "Pajoniiir-M1" (path "/2c8dd352-b7b8-4d9e-8f93-5dd43be2a100/31000008-6b2a-4a3a-8c91-000000000008" (reference "J3") (unit 1))))

Commit message: feat: establish board-first B8 pre-layout
Populate the live PCB with the complete schematic footprint/net set, preserve fail-closed mechanical gates, and isolate DSI506 as a qualified display profile. Add reproducible placement validation, ERC/BOM evidence, and synchronized project documentation.
Parts:
- J3: symbol Connector:USB_A -> Pajoniiir-M1:USB_A_M1
Changed lines of the file:
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@@
   )
   (symbol
-    (lib_id "Connector:USB_A") (at 184.785 59.69 0) (unit 1)
+    (lib_id "Pajoniiir-M1:USB_A_M1") (at 184.785 59.69 0) (unit 1)
     (exclude_from_sim no) (in_bom yes) (on_board yes) (dnp no)
     (property "Reference" "J3" (at 176.785 42.69 0) (effects (font (size 1.27 1.27))))
