File: hardware/Pajoniiir-M1/12_MICROSD.kicad_sch (KiCad schematic)
At the start: 23 parts, among them J7 microSD SOCKET TBD-MECH, U13 TPS22918DBVR

Commit message: mechanical: lock Molex microSD footprint
Parts:
- J7: value microSD SOCKET TBD-MECH -> 503398-1892; footprint (none) -> Pajoniiir-M1:Molex_503398-1892
Changed lines of the file:
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@@
     (exclude_from_sim no) (in_bom yes) (on_board yes) (dnp no)
     (property "Reference" "J7" (at 202.71 63.09 0) (effects (font (size 1.27 1.27))))
-    (property "Value" "microSD SOCKET TBD-MECH" (at 202.71 65.59 0) (effects (font (size 1.27 1.27))))
-    (property "Footprint" "" (at 219.71 85.09 0) (effects (font (size 1.27 1.27)) (hide yes)))
-    (property "Datasheet" "~" (at 219.71 85.09 0) (effects (font (size 1.27 1.27)) (hide yes)))
+    (property "Value" "503398-1892" (at 202.71 65.59 0) (effects (font (size 1.27 1.27))))
+    (property "Footprint" "Pajoniiir-M1:Molex_503398-1892" (at 219.71 85.09 0) (effects (font (size 1.27 1.27)) (hide yes)))
+    (property "Datasheet" "https://www.molex.com/content/dam/molex/molex-dot-com/products/automated/en-us/salesdrawingpdf/503/503398/5033981892_sd.pdf" (at 219.71 85.09 0) (effects (font (size 1.27 1.27)) (hide yes)))
     (pin "1") (pin "2") (pin "3") (pin "4")
     (pin "5") (pin "6") (pin "7") (pin "8")

Commit message: feat: establish board-first B8 pre-layout
Populate the live PCB with the complete schematic footprint/net set, preserve fail-closed mechanical gates, and isolate DSI506 as a qualified display profile. Add reproducible placement validation, ERC/BOM evidence, and synchronized project documentation.
Parts:
- J7: symbol Connector:Micro_SD_Card_Det1 -> Pajoniiir-M1:MicroSD_Det1_M1
Changed lines of the file:
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@@
   )
   (symbol
-    (lib_id "Connector:Micro_SD_Card_Det1") (at 219.71 85.09 0) (unit 1)
+    (lib_id "Pajoniiir-M1:MicroSD_Det1_M1") (at 219.71 85.09 0) (unit 1)
     (exclude_from_sim no) (in_bom yes) (on_board yes) (dnp no)
     (property "Reference" "J7" (at 202.71 63.09 0) (effects (font (size 1.27 1.27))))
